File: extras/schematics/power_meter.kicad_pcb (KiCad board)
At the start: 2 copper layers, 44.5 x 43.2 mm, 23 parts, among them J1 RF_UHF, J2 RF_SHF, J3 Conn_01x02, J4 Conn_01x04, U1 ltc5508, U2 ad8307

Commit message: Added missing files
Other:
- net class Default removed
